File: SoundBoxSTM32/audio.kicad_sch (KiCad schematic)
At the start: 3 parts, among them U2 DFR0299

Commit message: Added footprints, Ratsnest init
Parts:
- C40: footprint (none) -> Capacitor_SMD:C_0603_1608Metric
- U2: footprint Audio_Module:MODULE_DFR029_DFPLAYER -> Module:DFR0299
Changed lines of the file:
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@@
 			)
 		)
-		(property "Footprint" "Audio_Module:MODULE_DFR029_DFPLAYER"
+		(property "Footprint" "Module:DFR0299"
 			(at 149.86 92.71 0)
 			(hide yes)
@@
 			)
 		)
-		(property "Footprint" ""
+		(property "Footprint" "Capacitor_SMD:C_0603_1608Metric"
 			(at 188.9252 95.25 0)
 			(hide yes)
