File: SoundBoxSTM32/crystal.kicad_sch (KiCad schematic)
At the start: 6 parts, among them Y1 ECS-80-18-23B-JTN-TR

Commit message: Added footprints, Ratsnest init
Parts:
- C11, C12, C13, C14: footprint (none) -> Capacitor_SMD:C_0603_1608Metric
- XTAL1: footprint XTAL_SC32S-7PF20PPM_EPS -> Crystal:XTAL_SC32S-7PF20PPM_EPS
- Y1: footprint ECS-80-18-23B-JTN-TR:XTAL_ECS-80-18-23B-JTN-TR -> Crystal:XTAL_ECS-80-18-23B-JTN-TR
Changed lines of the file:
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@@
 			)
 		)
-		(property "Footprint" "ECS-80-18-23B-JTN-TR:XTAL_ECS-80-18-23B-JTN-TR"
+		(property "Footprint" "Crystal:XTAL_ECS-80-18-23B-JTN-TR"
 			(at 172.72 97.79 0)
 			(hide yes)
@@
 			)
 		)
-		(property "Footprint" ""
+		(property "Footprint" "Capacitor_SMD:C_0603_1608Metric"
 			(at 111.4552 106.68 0)
 			(hide yes)
@@
 			)
 		)
-		(property "Footprint" ""
+		(property "Footprint" "Capacitor_SMD:C_0603_1608Metric"
 			(at 199.0852 110.49 0)
 			(hide yes)
@@
 			)
 		)
-		(property "Footprint" "XTAL_SC32S-7PF20PPM_EPS"
+		(property "Footprint" "Crystal:XTAL_SC32S-7PF20PPM_EPS"
 			(at 93.98 96.52 0)
 			(hide yes)
@@
 			)
 		)
-		(property "Footprint" ""
+		(property "Footprint" "Capacitor_SMD:C_0603_1608Metric"
 			(at 150.8252 110.49 0)
 			(hide yes)
@@
 			)
 		)
-		(property "Footprint" ""
+		(property "Footprint" "Capacitor_SMD:C_0603_1608Metric"
 			(at 88.5952 106.68 0)
 			(hide yes)
