File: SoundBoxSTM32/power.kicad_sch (KiCad schematic)
At the start: 17 parts, among them J3 Barrel_Jack, Q1 PMOS, Q2 FS8205A, SW1 OS102011MA1QN1, U3 1043, U4 DW01A, U5 TPS3840PL35DBVR, U6 TLV75733PDBVR

Commit message: Added footprints, Ratsnest init
Parts:
- C21, C22, C23, C24, C25: footprint (none) -> Capacitor_SMD:C_0603_1608Metric
- D5: footprint Diode_SMD:SOD3715X145N -> Diode_SMD:1N5819HW-7-F
- J3: footprint (none) -> Connector_BarrelJack:BarrelJack_Horizontal
- Q1: footprint (none) -> Package_TO_SOT_SMD:SOT-23
- Q2: footprint FS8205A:SOP65P640X120-8N -> Transistor_Power:FS8205A
- R3, R4, R5: footprint (none) -> Resistor_SMD:R_0603_1608Metric
- SW1: footprint OS102011MA1QN1:SWITCH_11MA1QN1 -> Valve:OS102011MA1QN1
- U3: footprint 1043_KEY -> Battery:1043_KEY
- U5: footprint DBV0005A_N -> Filter:TPS3840PL42DBVR
- U6: footprint DBV0005A_N -> Battery:SOT95P280X145-5N_TLV75733PDBVR
Changed lines of the file:
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@@
 			)
 		)
-		(property "Footprint" ""
+		(property "Footprint" "Capacitor_SMD:C_0603_1608Metric"
 			(at 263.8552 59.69 0)
 			(hide yes)
@@
 			)
 		)
-		(property "Footprint" ""
+		(property "Footprint" "Capacitor_SMD:C_0603_1608Metric"
 			(at 249.8852 125.73 0)
 			(hide yes)
@@
 			)
 		)
-		(property "Footprint" ""
+		(property "Footprint" "Capacitor_SMD:C_0603_1608Metric"
 			(at 101.2952 140.97 0)
 			(hide yes)
@@
 			)
 		)
-		(property "Footprint" ""
+		(property "Footprint" "Resistor_SMD:R_0603_1608Metric"
 			(at 137.922 138.43 90)
 			(hide yes)
@@
 			)
 		)
-		(property "Footprint" ""
+		(property "Footprint" "Connector_BarrelJack:BarrelJack_Horizontal"
 			(at 66.04 56.896 0)
 			(hide yes)
@@
 			)
 		)
-		(property "Footprint" "Diode_SMD:SOD3715X145N"
+		(property "Footprint" "Diode_SMD:1N5819HW-7-F"
 			(at 86.36 53.34 0)
 			(hide yes)
@@
 			)
 		)
-		(property "Footprint" ""
+		(property "Footprint" "Capacitor_SMD:C_0603_1608Metric"
 			(at 195.2752 135.89 0)
 			(hide yes)
@@
 			)
 		)
-		(property "Footprint" "FS8205A:SOP65P640X120-8N"
+		(property "Footprint" "Transistor_Power:FS8205A"
 			(at 121.92 147.32 0)
 			(hide yes)
@@
 			)
 		)
-		(property "Footprint" "OS102011MA1QN1:SWITCH_11MA1QN1"
+		(property "Footprint" "Valve:OS102011MA1QN1"
 			(at 243.84 52.07 0)
 			(hide yes)
@@
 			)
 		)
-		(property "Footprint" "1043_KEY"
+		(property "Footprint" "Battery:1043_KEY"
 			(at 30.48 156.21 0)
 			(hide yes)
@@
 			)
 		)
-		(property "Footprint" "DBV0005A_N"
+		(property "Footprint" "Filter:TPS3840PL42DBVR"
 			(at 218.44 46.99 0)
 			(hide yes)
@@
 			)
 		)
-		(property "Footprint" ""
+		(property "Footprint" "Resistor_SMD:R_0603_1608Metric"
 			(at 43.942 128.27 90)
 			(hide yes)
@@
 			)
 		)
-		(property "Footprint" ""
+		(property "Footprint" "Capacitor_SMD:C_0603_1608Metric"
 			(at 188.9252 59.69 0)
 			(hide yes)
@@
 			)
 		)
-		(property "Footprint" "DBV0005A_N"
+		(property "Footprint" "Battery:SOT95P280X145-5N_TLV75733PDBVR"
 			(at 218.44 121.92 0)
 			(hide yes)
@@
 			)
 		)
-		(property "Footprint" ""
+		(property "Footprint" "Resistor_SMD:R_0603_1608Metric"
 			(at 121.92 110.998 90)
 			(hide yes)
@@
 			)
 		)
-		(property "Footprint" ""
+		(property "Footprint" "Package_TO_SOT_SMD:SOT-23"
 			(at 43.18 105.41 0)
 			(hide yes)
