File: SoundBoxSTM32/resetboot.kicad_sch (KiCad schematic)
At the start: 8 parts

Commit message: Added footprints, Ratsnest init
Parts:
- SWSW_CHIP_PU1, SW_GPIO1: footprint Button_Switch_SMD:SW_PTS810_SJM_250_SMTR_LFS -> Button_Switch_SMD:PTS810_SJM_250_SMTR_LFS
Changed lines of the file:
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@@
 			)
 		)
-		(property "Footprint" "Button_Switch_SMD:SW_PTS810_SJM_250_SMTR_LFS"
+		(property "Footprint" "Button_Switch_SMD:PTS810_SJM_250_SMTR_LFS"
 			(at 181.61 100.33 0)
 			(hide yes)
@@
 			)
 		)
-		(property "Footprint" "Button_Switch_SMD:SW_PTS810_SJM_250_SMTR_LFS"
+		(property "Footprint" "Button_Switch_SMD:PTS810_SJM_250_SMTR_LFS"
 			(at 95.25 91.44 0)
 			(hide yes)
