File: SoundBoxSTM32/SoundBoxSTM32.kicad_pcb (KiCad board)
At the start: 2 copper layers, 102 parts, among them J1 Conn_01x08, J2 Conn_01x05, J3 Barrel_Jack, Q1 PMOS, Q2 FS8205A, SW1 OS102011MA1QN1, SW10 SW_SPDT, SW2 SW_SPDT, SW3 SW_SPDT, SW4 SW_SPDT, SW5 SW_SPDT, SW6 SW_SPDT, SW7 SW_SPDT, SW8 SW_SPDT, SW9 SW_SPDT, U1 STM32H573RIT6, U2 DFR0299, U3 1043, U4 DW01A, U5 TPS3840PL35DBVR, U6 TLV75733PDBVR, Y1 ECS-80-18-23B-JTN-TR

Commit message: Rough organization of ratsnest
Parts:
- added H1: MountingHole_Pad, MountingHole:MountingHole_5.3mm_M5_DIN965_Pad, F.Cu at (206.0, 206.0)
- added H2: MountingHole_Pad, MountingHole:MountingHole_5.3mm_M5_DIN965_Pad, F.Cu at (206.0, 52.0)
- added H3: MountingHole_Pad, MountingHole:MountingHole_5.3mm_M5_DIN965_Pad, F.Cu at (52.0, 52.0)
- added H4: MountingHole_Pad, MountingHole:MountingHole_5.3mm_M5_DIN965_Pad, F.Cu at (52.0, 206.0)
- J1: value Conn_01x08 -> JTAG
- J2: value Conn_01x05 -> DEBUG
- U3: moved to B.Cu
- moved J2 283.2 mm to (63.8, 212.8), turned to 90 degrees
- moved J1 249.3 mm to (92.9, 212.9), turned to 90 degrees
- moved LED6 243.5 mm to (69.0, 201.8)
- moved STATUS_LED1 226.1 mm to (83.8, 211.9)
- moved U2 219.5 mm to (52.5, 178.0), turned to -90 degrees
- moved U3 219.2 mm to (57.1, 64.8), turned to 90 degrees
- moved Speaker1 215.4 mm to (72.0, 171.9), turned to 180 degrees
- moved U1 210.9 mm to (99.2, 159.1), turned to 180 degrees
- moved RESET 210.6 mm to (119.0, 212.9)
- moved BOOT 207.5 mm to (128.6, 212.9)
- moved LED7 199.7 mm to (129.1, 201.8)
- moved LED3 190.2 mm to (69.0, 138.0)
- moved SW1 188.5 mm to (44.0, 144.9), turned to -90 degrees
- moved SW4 180.5 mm to (183.6, 65.3)
- moved XTAL1 176.2 mm to (111.0, 162.8), turned to 180 degrees
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- renumbered SWSW_CHIP_PU1 to BOOT, SW_GPIO1 to RESET
Other:
- board outline added: 174 x 174 mm

Commit message: Base layout done, added image
Parts:
- added C41: 100nF, Capacitor_SMD:C_0603_1608Metric, F.Cu at (189.2, 143.2)
- added G***: LOGO, LOGO, F.Cu at (827.1, 200.0)
- J1: value JTAG -> Conn_01x08
- J2: value DEBUG -> Conn_01x05
- moved STATUS_LED1 163.2 mm to (65.5, 49.7)
- moved C32 108.9 mm to (69.1, 79.4)
- moved C40 101.6 mm to (66.0, 181.2)
- moved R11 100.0 mm to (75.1, 78.7), turned to 180 degrees
- moved C34 92.3 mm to (189.2, 79.3)
- moved C37 86.4 mm to (69.0, 206.9)
- moved R17 85.7 mm to (75.0, 142.5), turned to 180 degrees
- moved R15 84.2 mm to (195.1, 78.6), turned to 180 degrees
- moved C33 81.3 mm to (129.0, 79.2)
- moved R23 81.0 mm to (75.0, 206.4), turned to 180 degrees
- moved C35 80.1 mm to (69.0, 143.1)
- moved C23 72.5 mm to (61.6, 149.9)
- moved R5 70.9 mm to (64.4, 156.3), turned to 180 degrees
- moved R3 69.1 mm to (64.4, 162.6)
- moved R13 66.9 mm to (135.0, 78.6), turned to 180 degrees
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- renumbered BOOT to SWSW_CHIP_PU1, RESET to SW_GPIO1
Routing:
- net VCC_3V3: track 0.00 -> 1007.7 mm, vias 0 -> 7
- net Net-(LED5-DOUT): track 0.00 -> 241.8 mm
- net Net-(LED2-DOUT): track 0.00 -> 233.8 mm
- net Net-(STATUS_LED1-DIN): track 0.00 -> 180.5 mm, vias 0 -> 2
- net BAT+: track 0.00 -> 180.5 mm, vias 0 -> 4
- net GND: track 0.00 -> 172.6 mm, vias 0 -> 935
- net NRST: track 0.00 -> 171.5 mm, vias 0 -> 2
- net VSYS: track 0.00 -> 151.8 mm, vias 0 -> 1
- net Net-(SW4-B): track 0.00 -> 143.4 mm, vias 0 -> 2
- net Net-(SW2-B): track 0.00 -> 137.9 mm, vias 0 -> 1
- net BAT-: track 0.00 -> 118.0 mm, vias 0 -> 3
- net Net-(SW8-B): track 0.00 -> 105.0 mm
- net Net-(SW10-B): track 0.00 -> 100.2 mm, vias 0 -> 1
- net USART2_TX: track 0.00 -> 97.1 mm, vias 0 -> 1
- net Net-(SW3-B): track 0.00 -> 92.6 mm, vias 0 -> 1
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- added copper zone on B.Cu, net GND
- added copper zone on F.Cu, net GND
Other:
- outline, holes or cut-outs redrawn
- board text added: "SoundBox v1.0.0 08.10.2026 Dominik Neugebauer"
