File: SoundBoxSTM32/SoundBoxSTM32.kicad_pcb (KiCad board)
At the start: 2 copper layers, 174 x 174 mm, 108 parts, among them J1 Conn_01x08, J2 Conn_01x05, J3 Barrel_Jack, Q1 PMOS, Q2 FS8205A, SW1 OS102011MA1QN1, SW10 SW_SPDT, SW2 SW_SPDT, SW3 SW_SPDT, SW4 SW_SPDT, SW5 SW_SPDT, SW6 SW_SPDT, SW7 SW_SPDT, SW8 SW_SPDT, SW9 SW_SPDT, U1 STM32H573RIT6, U2 DFR0299, U3 1043, U4 DW01A, U5 TPS3840PL35DBVR, U6 TLV75733PDBVR, Y1 ECS-80-18-23B-JTN-TR

Commit message: Finished rough layout design
Parts:
- added H10: MountingHole, MountingHole:MountingHole_5.3mm_M5, F.Cu at (279.5, 83.0)
- added H11: MountingHole, MountingHole:MountingHole_5.3mm_M5, F.Cu at (244.5, 83.0)
- added H12: MountingHole, MountingHole:MountingHole_5.3mm_M5, F.Cu at (244.5, 48.0)
- added H13: MountingHole, MountingHole:MountingHole_5.3mm_M5, F.Cu at (222.5, 48.0)
- added H14: MountingHole, MountingHole:MountingHole_5.3mm_M5, F.Cu at (182.5, 48.0)
- added H15: MountingHole, MountingHole:MountingHole_5.3mm_M5, F.Cu at (222.5, 83.0)
- added H16: MountingHole, MountingHole:MountingHole_5.3mm_M5, F.Cu at (182.5, 83.0)
- added H17: MountingHole, MountingHole:MountingHole_5.3mm_M5, F.Cu at (125.5, 210.0)
- added H18: MountingHole, MountingHole:MountingHole_5.3mm_M5, F.Cu at (125.5, 175.0)
- added H19: MountingHole, MountingHole:MountingHole_5.3mm_M5, F.Cu at (160.5, 175.0)
- added H20: MountingHole, MountingHole:MountingHole_5.3mm_M5, F.Cu at (160.5, 210.0)
- added H21: MountingHole, MountingHole:MountingHole_5.3mm_M5, F.Cu at (182.5, 175.0)
- added H22: MountingHole, MountingHole:MountingHole_5.3mm_M5, F.Cu at (182.5, 210.0)
- added H23: MountingHole, MountingHole:MountingHole_5.3mm_M5, F.Cu at (222.5, 175.0)
- added H24: MountingHole, MountingHole:MountingHole_5.3mm_M5, F.Cu at (222.5, 210.0)
- added H25: MountingHole, MountingHole:MountingHole_5.3mm_M5, F.Cu at (244.5, 175.0)
- added H26: MountingHole, MountingHole:MountingHole_5.3mm_M5, F.Cu at (244.5, 210.0)
- added H27: MountingHole, MountingHole:MountingHole_5.3mm_M5, F.Cu at (279.5, 175.0)
- added H28: MountingHole, MountingHole:MountingHole_5.3mm_M5, F.Cu at (279.5, 210.0)
- added H29: MountingHole, MountingHole:MountingHole_5.3mm_M5, F.Cu at (125.5, 111.5)
- added H30: MountingHole, MountingHole:MountingHole_5.3mm_M5, F.Cu at (182.5, 111.5)
- added H31: MountingHole, MountingHole:MountingHole_5.3mm_M5, F.Cu at (244.5, 111.5)
- added H32: MountingHole, MountingHole:MountingHole_5.3mm_M5, F.Cu at (160.5, 146.5)
- added H33: MountingHole, MountingHole:MountingHole_5.3mm_M5, F.Cu at (222.5, 146.5)
- added H34: MountingHole, MountingHole:MountingHole_5.3mm_M5, F.Cu at (279.5, 146.5)
- added H35: MountingHole, MountingHole:MountingHole_5.3mm_M5, F.Cu at (160.5, 111.5)
- added H36: MountingHole, MountingHole:MountingHole_5.3mm_M5, F.Cu at (222.5, 111.5)
- added H37: MountingHole, MountingHole:MountingHole_5.3mm_M5, F.Cu at (279.5, 111.5)
- added H38: MountingHole, MountingHole:MountingHole_5.3mm_M5, F.Cu at (125.5, 146.5)
- added H39: MountingHole, MountingHole:MountingHole_5.3mm_M5, F.Cu at (182.5, 146.5)
- added H40: MountingHole, MountingHole:MountingHole_5.3mm_M5, F.Cu at (244.5, 146.5)
- added H5: MountingHole, MountingHole:MountingHole_5.3mm_M5, F.Cu at (125.5, 48.0)
- added H6: MountingHole, MountingHole:MountingHole_5.3mm_M5, F.Cu at (160.5, 48.0)
- added H7: MountingHole, MountingHole:MountingHole_5.3mm_M5, F.Cu at (160.5, 83.0)
- added H8: MountingHole, MountingHole:MountingHole_5.3mm_M5, F.Cu at (125.5, 83.0)
- added H9: MountingHole, MountingHole:MountingHole_5.3mm_M5, F.Cu at (279.5, 48.0)
- moved STATUS_LED1 265.8 mm to (304.0, 167.0), turned to 90 degrees
- moved J2 250.6 mm to (304.0, 103.5), turned to 180 degrees
- moved J1 224.6 mm to (304.0, 136.2), turned to 180 degrees
- moved SW_GPIO1 159.3 mm to (304.6, 154.7), turned to 90 degrees
- moved R6 155.2 mm to (300.1, 157.6), turned to 180 degrees
- moved SWSW_CHIP_PU1 154.4 mm to (304.6, 145.2), turned to 90 degrees
- moved R9 153.5 mm to (300.1, 154.7), turned to 180 degrees
- moved C15 151.9 mm to (300.1, 151.8), turned to 0 degrees
- moved R8 149.7 mm to (300.1, 147.8), turned to 180 degrees
- moved R7 148.3 mm to (300.1, 145.0), turned to 180 degrees
- moved C16 147.0 mm to (300.1, 142.2), turned to 0 degrees
- moved H1 93.5 mm to (299.5, 206.0)
- moved H2 93.5 mm to (299.5, 52.0)
- moved C34 73.5 mm to (262.7, 79.3)
- moved C41 73.5 mm to (262.7, 143.2)
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Routing:
- net Net-(LED0-DIN): track 29.2 -> 294.4 mm
- net BAT-: track 118.0 -> 368.7 mm, vias 3 -> 2
- net VSYS: track 151.8 -> 357.3 mm
- net BAT+: track 180.5 -> 341.7 mm, vias 4 -> 0
- net SWDIO: track 60.5 -> 138.9 mm, vias 1 -> 2
- net SWCLK: track 58.2 -> 134.0 mm, vias 1 -> 2
- net JTDI: track 64.3 -> 140.0 mm, vias 1 -> 2
- net NJTRST: track 71.9 -> 133.1 mm
- net Net-(STATUS_LED1-DIN): track 180.5 -> 122.5 mm
- net GND: track 208.6 -> 159.9 mm, vias 954 -> 904
- net BOOT0: track 77.4 -> 124.3 mm, vias 2 -> 4
- net NRST: track 163.8 -> 120.9 mm, vias 2 -> 5
- net SWO: track 86.6 -> 122.0 mm
- net USART2_RX: track 86.0 -> 109.6 mm
- net DFR_BUSY: track 73.0 -> 92.9 mm
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Other:
- board size 174 x 174 mm -> 214 x 174 mm
- board text added: "114mm"
- board text added: "149mm"
- board text added: "22mm"
- board text added: "30mm"
- board text added: "35mm"
- board text added: "6mm"
- board text added: "Debugger, JTAG, Buttons and LED on this side!"

Commit message: Fixed critical footprint error on PMOS
Parts:
- removed Q1: PMOS, Package_TO_SOT_SMD:SOT-23
- added Q3: AO3401A, Transformer_SMD:PMOS-SOT23-3, F.Cu at (117.3, 159.6)
- moved SWSW_CHIP_PU1 0.47 mm to (304.6, 144.7)
- moved SW_GPIO1 0.26 mm to (304.7, 155.0)
Routing:
- net VSYS: track 357.3 -> 377.3 mm, vias 1 -> 4
- net GND: track 159.9 -> 171.3 mm, vias 904 -> 899
- net BAT+: track 341.7 -> 351.0 mm, vias 0 -> 2
- net BAT-: track 368.7 -> 362.0 mm
- net Net-(SW4-B): track 146.1 -> 151.0 mm
- net JTDI: track 140.0 -> 137.1 mm
- net VBUS: track 13.3 -> 16.2 mm
- net Net-(SW7-B): track 85.3 -> 83.0 mm
- net Net-(U4-VCC): track 23.9 -> 25.8 mm
- net SWDIO: track 138.9 -> 140.7 mm
- net Net-(STATUS_LED1-DIN): track 122.5 -> 121.4 mm
- net NJTRST: track 133.1 -> 132.1 mm
- net SWCLK: track 134.0 -> 134.6 mm

Commit message: BOM done, evaluation done, schematic for cheaper version done
Parts:
- added R1: 100k, Resistor_SMD:R_0603_1608Metric, F.Cu at (131.4, 159.9)
- U5: value TPS3840PL35DBVR -> TPS3840DL35DBVR
Routing:
- net LDO_EN: track 25.4 -> 39.3 mm, vias 2 -> 4
- net VSYS: track 377.3 -> 382.2 mm
Other:
- board text added: "TODO: Kondensator von Buttons NRST & BOOT zum Chip (STM32)"
