File: SoundBoxSTM32/SoundBoxSTM32.kicad_sch (KiCad schematic)
At the start: 4 parts

Commit message: Finished rough layout design
Parts:
- added H10, H11, H12, H13, H14, H15, H16, H17, H18, H19, H20, H21, H22, H23, H24, H25, H26, H27, H28, H29, H30, H31, H32, H33, H34, H35, H36, H37, H38, H39, H40, H5, H6, H7, H8, H9: MountingHole, MountingHole:MountingHole_5.3mm_M5, symbol Mechanical:MountingHole
Other:
- moved on the sheet: H1, H2, H3, H4
