File: SoundBoxSTM32_cheap/audio.kicad_sch (KiCad schematic)
At the start: 3 parts, among them U2 DFR0299

Commit message: Finished layout for cheap version
Parts:
- C40: footprint Capacitor_SMD:C_0603_1608Metric -> Capacitor_SMD:C_1206_3216Metric_Pad1.33x1.80mm_HandSolder
Changed lines of the file:
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@@
 			)
 		)
-		(property "Footprint" "Capacitor_SMD:C_0603_1608Metric"
+		(property "Footprint" "Capacitor_SMD:C_1206_3216Metric_Pad1.33x1.80mm_HandSolder"
 			(at 182.5752 96.52 0)
 			(hide yes)
