File: SoundBoxSTM32_cheap/switches.kicad_sch (KiCad schematic)
At the start: 36 parts, among them SW11 SW_Push, SW12 SW_Push, SW13 SW_Push, SW14 SW_Push, SW15 SW_Push, SW16 SW_Push, SW17 SW_Push, SW18 SW_Push, SW19 SW_Push

Commit message: Finished layout for cheap version
Changed lines of the file:
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@@
 		(property "Value" "10k"
 			(at 147.32 45.466 90)
-			(hide yes)
 			(show_name no)
 			(do_not_autoplace no)
@@
 		(property "Value" "10k"
 			(at 147.32 82.296 90)
-			(hide yes)
 			(show_name no)
 			(do_not_autoplace no)
@@
 		(property "Value" "10k"
 			(at 83.82 119.126 90)
-			(hide yes)
 			(show_name no)
 			(do_not_autoplace no)
@@
 		(property "Value" "10k"
 			(at 147.32 119.126 90)
-			(hide yes)
 			(show_name no)
 			(do_not_autoplace no)
@@
 		(property "Value" "10k"
 			(at 83.82 82.296 90)
-			(hide yes)
 			(show_name no)
 			(do_not_autoplace no)
@@
 		(property "Value" "10k"
 			(at 83.82 45.466 90)
-			(hide yes)
 			(show_name no)
 			(do_not_autoplace no)
@@
 		(property "Value" "10k"
 			(at 210.82 45.466 90)
-			(hide yes)
-			(show_name no)
-			(do_not_autoplace no)
+			(show_name no)
+			(do_not_autoplace no)
