File: SoundBoxSTM32_cheap/stm32.kicad_sch (KiCad schematic)
At the start: 4 parts, among them J1 Conn_01x05, U1 STM32G030K8Tx

Commit message: Finished LoveBox, Finished Rubberducky
Connections:
- net BAT_SENSE: now reaches U1.17 (PB2)
- no-connect marks 10 -> 9
Changed lines of the file:
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@@
-	)
-	(no_connect
-		(at 115.57 118.11)
 	)
 	(no_connect
@@
 			)
 		)
+	)
+	(global_label "BAT_SENSE"
+		(shape input)
+		(at 115.57 118.11 180)
+		(fields_autoplaced yes)
+		(effects
+			(font
+				(size 1.27 1.27)
+			)
+			(justify right)
+		)
+		(property "Intersheetrefs" "${INTERSHEET_REFS}"
+			(at 102.2435 118.11 0)
+			(hide yes)
+			(show_name no)
+			(do_not_autoplace no)
+			(effects
+				(font
+					(size 1.27 1.27)
+				)
+				(justify right)
+			)
+		)
