File: SoundBoxSTM32_cheap/SoundBoxSTM32_cheap.kicad_pcb (KiCad board)
At the start: 2 copper layers, 154.1 x 125.9 mm, 140 parts, among them J1 Conn_01x05, Q2 FS8205A, Q3 AO3401A, SW1 OS102011MA1QN1, SW11 SW_Push, SW12 SW_Push, SW13 SW_Push, SW14 SW_Push, SW15 SW_Push, SW16 SW_Push, SW17 SW_Push, SW18 SW_Push, SW19 SW_Push, U1 STM32G030K8Tx, U10 WS2812B, U11 WS2812B, U12 WS2812B, U13 WS2812B, U14 WS2812B, U15 WS2812B, U16 WS2812B, U2 DFR0299, U3 1043, U4 DW01A, U5 TPS3840DL35DBVR, U6 TLV75733PDBVR, U7 WS2812B, U8 WS2812B, U9 WS2812B

Commit message: Finished layout for cheap version
Parts:
- removed C32, C33, C34, C35, C36, C37, C38, C39, C41: 100nF, Capacitor_SMD:C_0603_1608Metric
- removed R28: 330, Resistor_SMD:R_0603_1608Metric
- added G***: LOGO, LOGO, F.Cu at (426.1, 192.1)
- U3: moved to B.Cu
- moved Speaker1 201.1 mm to (15.8, 165.3), turned to 90 degrees
- moved R30 192.2 mm to (48.8, 167.6), turned to 180 degrees
- moved C40 175.0 mm to (37.8, 155.6), turned to 180 degrees
- moved U2 173.9 mm to (24.1, 151.2), turned to -90 degrees
- moved R42 173.5 mm to (48.8, 104.0), turned to 180 degrees
- moved H1 172.8 mm to (22.9, 176.1)
- moved U3 160.1 mm to (25.3, 32.6), turned to 90 degrees
- moved R32 159.2 mm to (48.9, 40.5), turned to 180 degrees
- moved R44 152.7 mm to (108.6, 167.7), turned to 180 degrees
- moved SW11 146.0 mm to (63.0, 158.0)
- moved C17 143.5 mm to (48.9, 42.4)
- moved SW17 138.6 mm to (63.0, 94.5)
- moved H2 132.9 mm to (22.9, 22.2)
- moved U13 127.8 mm to (60.5, 174.2), turned to 180 degrees
- moved C50 123.9 mm to (110.0, 132.8), turned to 180 degrees
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Routing:
- net VCC_3V3: track 0.00 -> 969.5 mm, vias 0 -> 22
- net RE0: track 0.00 -> 202.9 mm
- net RE1: track 0.00 -> 202.3 mm
- net Net-(U7-DIN): track 0.00 -> 197.5 mm, vias 0 -> 4
- net Net-(R32-Pad1): track 0.00 -> 194.3 mm, vias 0 -> 3
- net Net-(R36-Pad1): track 0.00 -> 153.0 mm, vias 0 -> 3
- net GND: track 0.00 -> 138.2 mm, vias 0 -> 49
- net Net-(R34-Pad1): track 0.00 -> 132.4 mm, vias 0 -> 1
- net SWDIO: track 0.00 -> 129.4 mm
- net SWCLK: track 0.00 -> 126.1 mm
- net Net-(R30-Pad1): track 0.00 -> 119.5 mm, vias 0 -> 2
- net Net-(R46-Pad1): track 0.00 -> 114.8 mm, vias 0 -> 3
- net NRST: track 0.00 -> 113.8 mm
- net DFR_BUSY: track 0.00 -> 107.5 mm, vias 0 -> 3
- net Net-(R42-Pad1): track 0.00 -> 107.4 mm, vias 0 -> 4
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- added copper zone on B.Cu, net GND
- added copper zone on F.Cu, net GND
Other:
- board size 154.1 x 125.9 mm -> 214 x 174 mm
- board text added: "SoundBox v1.0.0 08.10.2026 Dominik Neugebauer"

Commit message: Finished LoveBox, Finished Rubberducky
Parts:
- added C32: 100nF, Capacitor_SMD:C_0603_1608Metric, F.Cu at (113.4, 131.0)
- added R10: 100k, Resistor_SMD:R_0603_1608Metric, F.Cu at (113.4, 127.5)
- added R9: 100k, Resistor_SMD:R_0603_1608Metric, F.Cu at (113.4, 129.2)
- C40: footprint Capacitor_SMD:C_0603_1608Metric -> Capacitor_SMD:C_1206_3216Metric_Pad1.33x1.80mm_HandSolder
- moved G*** 524.8 mm to (949.3, 232.5)
- moved C40 4.93 mm to (38.1, 160.5)
- moved H11 2.50 mm to (102.4, 18.6)
- moved H12 2.50 mm to (102.4, 53.6)
- moved H13 2.50 mm to (137.4, 53.6)
- moved H14 2.50 mm to (137.4, 18.6)
- moved H18 2.50 mm to (137.4, 82.1)
- moved H20 2.50 mm to (137.4, 117.1)
- moved H21 2.50 mm to (102.4, 145.6)
- moved H22 2.50 mm to (102.4, 180.6)
- moved H27 2.50 mm to (137.4, 145.6)
- moved H28 2.50 mm to (137.4, 180.6)
- moved H29 2.50 mm to (102.4, 82.1)
- moved H31 2.50 mm to (102.4, 117.1)
Connections:
- U1 pad 17: unconnected-(U1-PB2-Pad17) -> BAT_SENSE
Routing:
- net BAT+: track 100.7 -> 214.3 mm, vias 1 -> 2
- net GND: track 138.2 -> 150.3 mm, vias 49 -> 1050
- net BAT_SENSE: track 0.00 -> 6.61 mm
- net VCC_3V3: track 969.5 -> 973.6 mm
- net Net-(R34-Pad1): track 132.4 -> 133.4 mm

Commit message: finished
Parts:
- moved G*** 526.7 mm to (423.0, 211.6)
Changed lines of the file:
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@@
 	(footprint "LOGO"
 		(layer "F.Cu")
-		(at 949.275 232.525)
+		(at 423.01 211.63)
 		(property "Reference" "G***"
 			(at 0 0 0)
@@
 	)
 	(segment
+		(start 115.115 131.965)
+		(end 114.15 131)
+		(width 0.2)
+		(layer "F.Cu")
+		(net "BAT_SENSE")
+	)
+	(segment
+		(start 114.15 131)
+		(end 114.15 129.25)
+		(width 0.2)
+		(layer "F.Cu")
+		(net "BAT_SENSE")
+	)
+	(segment
+		(start 114.15 129.25)
+		(end 114.2 129.2)
+		(width 0.2)
+		(layer "F.Cu")
+		(net "BAT_SENSE")
+	)
+	(segment
+		(start 116.785 131.965)
+		(end 115.115 131.965)
+		(width 0.2)
+		(layer "F.Cu")
+		(net "BAT_SENSE")
+	)
+	(segment
+		(start 114.2 129.2)
+		(end 114.2 127.45)
+		(width 0.2)
+		(layer "F.Cu")
+		(net "BAT_SENSE")
+	)
+	(segment
 		(start 109.175 105.87)
 		(end 115.08 105.87)
@@
 		(net "Net-(R7-Pad1)")
 	)
-	(segment
-		(start 115.115 131.965)
-		(end 114.15 131)
-		(width 0.2)
-		(layer "F.Cu")
-		(net "BAT_SENSE")
-	)
-	(segment
-		(start 114.15 131)
-		(end 114.15 129.25)
-		(width 0.2)
-		(layer "F.Cu")
-		(net "BAT_SENSE")
-	)
-	(segment
-		(start 114.15 129.25)
-		(end 114.2 129.2)
-		(width 0.2)
-		(layer "F.Cu")
-		(net "BAT_SENSE")
-	)
-	(segment
-		(start 116.785 131.965)
-		(end 115.115 131.965)
-		(width 0.2)
-		(layer "F.Cu")
-		(net "BAT_SENSE")
-	)
-	(segment
-		(start 114.2 129.2)
-		(end 114.2 127.45)
-		(width 0.2)
-		(layer "F.Cu")
-		(net "BAT_SENSE")
-	)
 	(zone
